Commit message: 初步完成，但是有bug

File: urdf/ur5_robotiq_85.urdf (robot description, URDF)
Before this commit: robot ur5_robotiq_85, 8 links, 7 joints
Links:
- added link camera_link, mass 0.01; visual box size=0.02 0.02 0.02
- added link gripper_tip_link
- added link robotiq_85_base_link, mass 0.636951; collision mesh filename=../meshes/robotiq_85/collision/robotiq_arg2f_85_base_link.s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; visual mesh filename=../meshes/robotiq_85/visual/robotiq_arg2f_85_base_link.dae
- added link robotiq_85_left_inner_finger, mass 0.019555; collision mesh filename=../meshes/robotiq_85/collision/robotiq_arg2f_85_inner_finge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; visual mesh filename=../meshes/robotiq_85/visual/robotiq_arg2f_85_inner_finger.d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
- added link robotiq_85_left_inner_knuckle, mass 0.029951; collision mesh filename=../meshes/robotiq_85/collision/robotiq_arg2f_85_inner_knuck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; visual mesh filename=../meshes/robotiq_85/visual/robotiq_arg2f_85_inner_knuckle.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
- added link robotiq_85_left_outer_finger, mass 0.027309; collision mesh filename=../meshes/robotiq_85/collision/robotiq_arg2f_85_outer_finge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; visual mesh filename=../meshes/robotiq_85/visual/robotiq_arg2f_85_outer_finger.d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
- added link robotiq_85_left_outer_knuckle, mass 0.018491; collision mesh filename=../meshes/robotiq_85/collision/robotiq_arg2f_85_outer_knuck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; visual mesh filename=../meshes/robotiq_85/visual/robotiq_arg2f_85_outer_knuckle.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
- added link robotiq_85_right_inner_finger, mass 0.019555; collision mesh filename=../meshes/robotiq_85/collision/robotiq_arg2f_85_inner_finge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; visual mesh filename=../meshes/robotiq_85/visual/robotiq_arg2f_85_inner_finger.d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
- added link robotiq_85_right_inner_knuckle, mass 0.029951; collision mesh filename=../meshes/robotiq_85/collision/robotiq_arg2f_85_inner_knuck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; visual mesh filename=../meshes/robotiq_85/visual/robotiq_arg2f_85_inner_knuckle.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
- added link robotiq_85_right_outer_finger, mass 0.027309; collision mesh filename=../meshes/robotiq_85/collision/robotiq_arg2f_85_outer_finge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; visual mesh filename=../meshes/robotiq_85/visual/robotiq_arg2f_85_outer_finger.d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
- added link robotiq_85_right_outer_knuckle, mass 0.018491; collision mesh filename=../meshes/robotiq_85/collision/robotiq_arg2f_85_outer_knuck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; visual mesh filename=../meshes/robotiq_85/visual/robotiq_arg2f_85_outer_knuckle.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
Joints:
- added joint camera_joint: type fixed, parent robotiq_85_base_link, child camera_link, origin xyz=0.0 0.0 -0.05 rpy=0.0 1.57079632679 0.0
- added joint finger_joint: type revolute, parent robotiq_85_base_link, child robotiq_85_left_outer_knuckle, origin xyz=-0.0306011 0.0 0.054904 rpy=0.0 0.0 0.0, axis 0 1 0, limit lower=0.0 upper=0.8 effort=50 velocity=0.5
- added joint gripper_tip_joint: type fixed, parent robotiq_85_base_link, child gripper_tip_link, origin xyz=0.0 0.0 0.145 rpy=0.0 0.0 0.0
- added joint left_inner_finger_joint: type revolute, parent robotiq_85_left_outer_knuckle, child robotiq_85_left_inner_finger, origin xyz=0.0 0.0 0.09585 rpy=0.0 0.0 0.0, axis 0 1 0, limit lower=-0.8 upper=0.0 effort=50 velocity=0.5, mimic joint=finger_joint multiplier=-1 offset=0
- added joint left_inner_knuckle_joint: type revolute, parent robotiq_85_base_link, child robotiq_85_left_inner_knuckle, origin xyz=-0.0127 0.0 0.06142 rpy=0.0 0.0 0.0, axis 0 1 0, limit lower=0.0 upper=0.8 effort=50 velocity=0.5, mimic joint=finger_joint multiplier=1 offset=0
- added joint left_outer_finger_joint: type fixed, parent robotiq_85_left_outer_knuckle, child robotiq_85_left_outer_finger, origin xyz=0.0 0.0 0.0 rpy=0.0 0.0 0.0
- added joint right_inner_finger_joint: type revolute, parent robotiq_85_right_outer_knuckle, child robotiq_85_right_inner_finger, origin xyz=0.0 0.0 0.09585 rpy=0.0 0.0 0.0, axis 0 1 0, limit lower=-0.8 upper=0.0 effort=50 velocity=0.5, mimic joint=finger_joint multiplier=-1 offset=0
- added joint right_inner_knuckle_joint: type revolute, parent robotiq_85_base_link, child robotiq_85_right_inner_knuckle, origin xyz=0.0127 0.0 0.06142 rpy=0.0 3.14159265359 0.0, axis 0 1 0, limit lower=0.0 upper=0.8 effort=50 velocity=0.5, mimic joint=finger_joint multiplier=1 offset=0
- added joint right_outer_finger_joint: type fixed, parent robotiq_85_right_outer_knuckle, child robotiq_85_right_outer_finger, origin xyz=0.0 0.0 0.0 rpy=0.0 0.0 0.0
- added joint right_outer_knuckle_joint: type revolute, parent robotiq_85_base_link, child robotiq_85_right_outer_knuckle, origin xyz=0.0306011 0.0 0.054904 rpy=0.0 3.14159265359 0.0, axis 0 1 0, limit lower=0.0 upper=0.8 effort=50 velocity=0.5, mimic joint=finger_joint multiplier=1 offset=0
- added joint robotiq_85_base_joint: type fixed, parent ee_link, child robotiq_85_base_link, origin xyz=0.0 0.0 0.0 rpy=0.0 0.0 0.0

Commit message: 修复了模型显示问题

File: urdf/ur5_robotiq_85.urdf (robot description, URDF)
Before this commit: robot ur5_robotiq_85, 19 links, 18 joints
Links:
- link robotiq_85_base_link: geometry collision mesh filename=../meshes/robotiq_85/collision/robotiq_arg2f_85_base_link.s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; visual mesh filename=../meshes/robotiq_85/visual/robotiq_arg2f_85_base_link.dae scale=0.001 0.001 0.001
- link robotiq_85_left_inner_finger: geometry collision mesh filename=../meshes/robotiq_85/collision/robotiq_arg2f_85_inner_finge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 scale=0.001 0.001 0.001; visual mesh filename=../meshes/robotiq_85/visual/robotiq_arg2f_85_inner_finger.d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 scale=0.001 0.001 0.001
- link robotiq_85_left_inner_knuckle: geometry collision mesh filename=../meshes/robotiq_85/collision/robotiq_arg2f_85_inner_knuck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 scale=0.001 0.001 0.001; visual mesh filename=../meshes/robotiq_85/visual/robotiq_arg2f_85_inner_knuckle.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 scale=0.001 0.001 0.001
- link robotiq_85_left_outer_finger: geometry collision mesh filename=../meshes/robotiq_85/collision/robotiq_arg2f_85_outer_finge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 scale=0.001 0.001 0.001; visual mesh filename=../meshes/robotiq_85/visual/robotiq_arg2f_85_outer_finger.d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 scale=0.001 0.001 0.001
- link robotiq_85_left_outer_knuckle: geometry collision mesh filename=../meshes/robotiq_85/collision/robotiq_arg2f_85_outer_knuck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 scale=0.001 0.001 0.001; visual mesh filename=../meshes/robotiq_85/visual/robotiq_arg2f_85_outer_knuckle.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 scale=0.001 0.001 0.001
- link robotiq_85_right_inner_finger: geometry collision mesh filename=../meshes/robotiq_85/collision/robotiq_arg2f_85_inner_finge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 scale=0.001 0.001 0.001; visual mesh filename=../meshes/robotiq_85/visual/robotiq_arg2f_85_inner_finger.d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 scale=0.001 0.001 0.001
- link robotiq_85_right_inner_knuckle: geometry collision mesh filename=../meshes/robotiq_85/collision/robotiq_arg2f_85_inner_knuck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 scale=0.001 0.001 0.001; visual mesh filename=../meshes/robotiq_85/visual/robotiq_arg2f_85_inner_knuckle.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 scale=0.001 0.001 0.001
- link robotiq_85_right_outer_finger: geometry collision mesh filename=../meshes/robotiq_85/collision/robotiq_arg2f_85_outer_finge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 scale=0.001 0.001 0.001; visual mesh filename=../meshes/robotiq_85/visual/robotiq_arg2f_85_outer_finger.d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 scale=0.001 0.001 0.001
- link robotiq_85_right_outer_knuckle: geometry collision mesh filename=../meshes/robotiq_85/collision/robotiq_arg2f_85_outer_knuck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 scale=0.001 0.001 0.001; visual mesh filename=../meshes/robotiq_85/visual/robotiq_arg2f_85_outer_knuckle.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 scale=0.001 0.001 0.001
